File: hardware/attinier85-light-sensor-shield-mk-1.0.brd (EAGLE design)
At the start: 36 x 25 mm, 9 parts, among them U1 ATTINIEST85_SHIELDV2

Commit message: renaming parts
Parts:
- U1: value ATTINIEST85_SHIELDV2 -> ATTINIER85_SHIELDV2; device A_butts:ATTINIEST85_SHIELD_V2 -> A_butts:ATTINIER85_SHIELD_V2
Changed lines of the file:
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@@
 <attribute name="DESIGNER" value="Nobody" x="13.97" y="-1.27" size="1.778" layer="27" display="off"/>
 </element>
-<element name="U1" library="A_butts" package="ATTINIEST85_SHIELD_V2" value="ATTINIEST85_SHIELDV2" x="18" y="12.5"/>
+<element name="U1" library="A_butts" package="ATTINIER85_SHIELD_V2" value="ATTINIER85_SHIELDV2" x="18" y="12.5"/>
 <element name="DISPLAY1" library="A_butts" package="ADAFRUIT_128X32_OLED_I2C_CLOSER_NOHOLES" value="Adafruit 128x32 OLED" x="18" y="2.5" smashed="yes"/>
 <element name="R1" library="A_butts" package="RESISTOR-AXIAL-PTH-7.62MM" value="4.7k" x="7" y="13" rot="MR90"/>
