File: hardware/attinier85-motherboard-mk-3.1.brd (EAGLE design)
At the start: 36 x 25 mm, 15 parts, among them IC1 Tiny85, IC2 LM2931, U1 ATTINIEST85_SHIELDV2

Commit message: renaming parts
Parts:
- U1: value ATTINIEST85_SHIELDV2 -> ATTINIER85_SHIELDV2; device A_butts:ATTINIEST85_SHIELD_V2 -> A_butts:ATTINIER85_SHIELD_V2
Changed lines of the file:
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@@
 <attribute name="VALUE" x="11.35" y="2.5" size="0.6" layer="21" font="vector" ratio="11" rot="R90" align="bottom-center"/>
 </element>
-<element name="U1" library="A_butts" package="ATTINIEST85_SHIELD_V2" value="ATTINIEST85_SHIELDV2" x="18" y="12.5"/>
+<element name="U1" library="A_butts" package="ATTINIER85_SHIELD_V2" value="ATTINIER85_SHIELDV2" x="18" y="12.5"/>
 </elements>
 <signals>
