File: hardware/attinier85-display-shield-mk-1.0.brd (EAGLE design)
At the start: 36 x 25 mm, 5 parts, among them U1 ATTINIER85_SHIELDV2

Commit message: cleaning up version spoo
Parts:
- added I2C: M04PTH, A_butts:1X04-PTH-VERT
- moved DISPLAY1 3.50 mm to (18.0, 2.50)
Connections:
- net GND: now also I2C.1
- net SCL: now also I2C.4
- net SDA: now also I2C.3
- net VCC: now also I2C.2
Routing:
- net SDA: track 30.2 -> 46.7 mm, vias 1 -> 2
- net SCL: track 32.9 -> 44.6 mm
- net VCC: track 39.9 -> 49.9 mm
- net DISP_RST: track 19.8 -> 23.3 mm
Changed lines of the file:
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@@
 <wire x1="33" y1="25" x2="3" y2="25" width="0" layer="20"/>
 <wire x1="3" y1="25" x2="0" y2="22" width="0" layer="20" curve="90"/>
-<text x="29" y="2" size="0.6" layer="21" font="vector" ratio="12" align="bottom-center">&gt;VERSION</text>
-<text x="29" y="2" size="0.6" layer="22" font="vector" ratio="12" rot="MR0" align="bottom-center">&gt;VERSION</text>
+<text x="27.5" y="22.5" size="1" layer="21" font="vector" ratio="16" align="center">&gt;VERSION</text>
+<text x="27.5" y="22.5" size="1" layer="22" font="vector" ratio="16" rot="MR0" align="center">&gt;VERSION</text>
 <text x="18" y="17.5" size="0.8" layer="22" font="vector" ratio="12" rot="MR0" align="bottom-center">&gt;AUTHOR</text>
 <text x="18" y="19" size="1" layer="22" font="vector" ratio="12" rot="MR0" align="bottom-center">ATTinier85 Display Shield</text>
-<text x="18" y="19" size="1" layer="21" font="vector" ratio="12" align="bottom-center">ATTinier85 Display Shield</text>
-<text x="18" y="17.5" size="0.8" layer="21" font="vector" ratio="12" align="bottom-center">&gt;AUTHOR</text>
+<text x="18" y="14" size="1" layer="21" font="vector" ratio="12" align="bottom-center">ATTinier85 Display Shield</text>
+<text x="18" y="11" size="0.8" layer="21" font="vector" ratio="12" align="bottom-center">&gt;AUTHOR</text>
+<text x="27.5" y="22.5" size="1" layer="1" font="vector" ratio="16" align="center">&gt;VERSION</text>
+<text x="27.5" y="22.5" size="1" layer="16" font="vector" ratio="16" rot="MR0" align="center">&gt;VERSION</text>
 </plain>
 <attributes>
@@
 </element>
 <element name="U1" library="A_butts" package="ATTINIER85_SHIELD_V2" value="ATTINIER85_SHIELDV2" x="18" y="12.5"/>
-<element name="DISPLAY1" library="A_butts" package="ADAFRUIT_128X32_OLED_I2C_CLOSER_NOHOLES" value="Adafruit 128x32 OLED" x="18" y="6" smashed="yes"/>
+<element name="DISPLAY1" library="A_butts" package="ADAFRUIT_128X32_OLED_I2C_CLOSER_NOHOLES" value="Adafruit 128x32 OLED" x="18" y="2.5" smashed="yes"/>
 <element name="R1" library="A_butts" package="RESISTOR-AXIAL-PTH-7.62MM" value="4.7k" x="7" y="13" rot="MR90"/>
 <element name="R2" library="A_butts" package="RESISTOR-AXIAL-PTH-7.62MM" value="4.7k" x="10" y="13" rot="MR90"/>
+<element name="I2C" library="A_butts" package="1X04-PTH-VERT" value="M04PTH" x="14.19" y="23.25" smashed="yes">
+<attribute name="NAME" x="12.69" y="23.25" size="1" layer="25" font="vector" ratio="12" rot="R90" align="bottom-center"/>
+</element>
 </elements>
 <signals>
@@
 <contactref element="U1" pad="GND@1"/>
 <contactref element="DISPLAY1" pad="GND"/>
+<contactref element="I2C" pad="1"/>
 </signal>
 <signal name="VCC">
 <contactref element="U1" pad="VCC"/>
 <contactref element="DISPLAY1" pad="VIN"/>
-<wire x1="24.35" y1="6" x2="24.35" y2="13.35" width="0.5" layer="1"/>
-<wire x1="24.35" y1="13.35" x2="28.56" y2="17.56" width="0.5" layer="1"/>
+<wire x1="24.35" y1="2.5" x2="24.35" y2="13.35" width="0.5" layer="1"/>
+<wire x1="24.35" y1="13.35" x2="28.5" y2="17.5" width="0.5" layer="1"/>
+<wire x1="28.5" y1="17.5" x2="28.56" y2="17.56" width="0.5" layer="1"/>
 <wire x1="28.56" y1="17.56" x2="33.25" y2="17.56" width="0.5" layer="1"/>
 <contactref element="R2" pad="P$2"/>
 <contactref element="R1" pad="P$2"/>
 <wire x1="7" y1="16.81" x2="10" y2="16.81" width="0.25" layer="1"/>
-<wire x1="10" y1="16.81" x2="27.81" y2="16.81" width="0.25" layer="1"/>
-<wire x1="27.81" y1="16.81" x2="28.56" y2="17.56" width="0.25" layer="1"/>
+<wire x1="27.81" y1="16.81" x2="28.5" y2="17.5" width="0.25" layer="1"/>
+<contactref element="I2C" pad="2"/>
+<wire x1="16.73" y1="18.04" x2="15.5" y2="16.81" width="0.25" layer="1"/>
+<wire x1="15.5" y1="16.81" x2="10" y2="16.81" width="0.25" layer="1"/>
+<wire x1="16.73" y1="18.04" x2="16.73" y2="23.25" width="0.25" layer="1"/>
+<wire x1="16.73" y1="18.04" x2="27.96" y2="18.04" width="0.25" layer="1"/>
+<wire x1="27.96" y1="18.04" x2="28.5" y2="17.5" width="0.25" layer="1"/>
 </signal>
 <signal name="SDA">
@@
 <wire x1="33.25" y1="9.94" x2="21.06" y2="9.94" width="0.25" layer="16"/>
 <via x="21.06" y="9.94" extent="1-16" drill="0.3302"/>
-<wire x1="21.06" y1="9.94" x2="13.94" y2="9.94" width="0.25" layer="1"/>
-<wire x1="13.94" y1="9.94" x2="11.65" y2="7.65" width="0.25" layer="1"/>
-<wire x1="11.65" y1="7.65" x2="11.65" y2="6" width="0.25" layer="1"/>
 <contactref element="R1" pad="P$1"/>
-<wire x1="7" y1="9.19" x2="10.19" y2="6" width="0.25" layer="1"/>
-<wire x1="10.19" y1="6" x2="11.65" y2="6" width="0.25" layer="1"/>
+<wire x1="7" y1="9.19" x2="11.65" y2="4.54" width="0.25" layer="1"/>
+<wire x1="11.65" y1="4.54" x2="11.65" y2="2.5" width="0.25" layer="1"/>
+<wire x1="21.06" y1="9.94" x2="17.05" y2="9.94" width="0.25" layer="1"/>
+<wire x1="17.05" y1="9.94" x2="11.65" y2="4.54" width="0.25" layer="1"/>
+<contactref element="I2C" pad="3"/>
+<wire x1="19.27" y1="23.25" x2="19.27" y2="16.5" width="0.25" layer="16"/>
+<via x="19.27" y="16.5" extent="1-16" drill="0.3302"/>
+<wire x1="19.27" y1="16.5" x2="19.27" y2="12.16" width="0.25" layer="1"/>
+<wire x1="19.27" y1="12.16" x2="17.05" y2="9.94" width="0.25" layer="1"/>
 </signal>
 <signal name="SCL">
 <contactref element="U1" pad="2"/>
 <contactref element="DISPLAY1" pad="SCL"/>
-<wire x1="33.25" y1="15.02" x2="16.02" y2="15.02" width="0.25" layer="16"/>
+<wire x1="21.81" y1="15.02" x2="16.02" y2="15.02" width="0.25" layer="16"/>
 <wire x1="16.02" y1="15.02" x2="14.19" y2="13.19" width="0.25" layer="16"/>
-<wire x1="14.19" y1="13.19" x2="14.19" y2="6" width="0.25" layer="16"/>
+<wire x1="14.19" y1="13.19" x2="14.19" y2="2.5" width="0.25" layer="16"/>
 <contactref element="R2" pad="P$1"/>
 <wire x1="14.19" y1="13.19" x2="10.19" y2="9.19" width="0.25" layer="16"/>
 <wire x1="10.19" y1="9.19" x2="10" y2="9.19" width="0.25" layer="16"/>
+<contactref element="I2C" pad="4"/>
+<wire x1="21.81" y1="23.25" x2="21.81" y2="15.02" width="0.25" layer="16"/>
+<wire x1="21.81" y1="15.02" x2="33.25" y2="15.02" width="0.25" layer="16"/>
 </signal>
 <signal name="DISP_RST">
@@
 <wire x1="2.75" y1="12.48" x2="15.52" y2="12.48" width="0.25" layer="1"/>
 <wire x1="15.52" y1="12.48" x2="16.73" y2="11.27" width="0.25" layer="16"/>
-<wire x1="16.73" y1="11.27" x2="16.73" y2="6" width="0.25" layer="16"/>
+<wire x1="16.73" y1="11.27" x2="16.73" y2="2.5" width="0.25" layer="16"/>
 <via x="15.52" y="12.48" extent="1-16" drill="0.3302"/>
 </signal>
