File: hardware/attinier85-motherboard-mk-1.0.sch (EAGLE design)
At the start: 17 parts, among them IC1 Tiny85

Commit message: cleaning up version spoo
Parts:
- removed H1, H2, H3, H4: HOLE#2, A_butts:HOLE#2
- removed JP1, JP2: (no value), A_butts:M05PTH
- removed MIC5235: V_REG_MIC5235, A_butts:V_REG_MIC5235
- added D1: 1N4001, A_butts:DIODEPTH-10.68MM
- added IC2: LM2931, A_butts:V_REG_78XXTO-92-INLINE
- added TVS1: 12V, A_butts:TVSDO-41-TVS-BIDIRECTIONAL
- added U1: ATTINIER85_SHIELDV2, A_butts:ATTINIER85_SHIELDV2
- C1: value 1uF -> 0.1uF; device A_butts:CAPACITOR-CERAMICC0603 -> A_butts:CAPACITOR-CERAMIC025-024X044
- C2: value 1uF -> 10uF; device A_butts:CAPACITOR-CERAMICC0805 -> A_butts:CAPACITOR-POLARIZEDE2.5-5
- C3: value 10uF -> 100uF; device A_butts:CAPACITOR-CERAMICC0805 -> A_butts:CAPACITOR-POLARIZEDE2.5-5
- IC1: device A_butts:ATTINY45TINY85-20-SMT -> A_butts:ATTINY45TINY85-20-DIP
- POWER: value LED0603 -> LED3MM-LESS; device A_butts:LED0603 -> A_butts:LED3MM-LESS
- R1, R2: device A_butts:RESISTORR0603 -> A_butts:RESISTORPTH-AXIAL-7.62MM
- RESET: value SPST-NO-TACTB3U-1000P -> DTS-6MM; device A_butts:SPST-NO-TACTB3U-1000P -> A_butts:SPST-NO-TACT3MM-PTH-SMALL-PADS
Connections:
- removed net D0: AVR_ISP.4, IC1.PB0(MOSI), JP2.1
- removed net D1: AVR_ISP.1, IC1.PB1(MISO), JP2.2
- removed net D2: AVR_ISP.3, IC1.PB2(SCK/ADC1), JP2.3
- new net MISO: AVR_ISP.MISO, IC1.PB1(MISO), U1.P1
- new net MOSI/SDA: AVR_ISP.MOSI, IC1.PB0(MOSI), U1.P0
- new net N$3: C2.+, D1.C, IC2.IN
- new net SCK/SCL: AVR_ISP.SCK, IC1.PB2(SCK/ADC1), U1.P2
- net D3: now also U1.P4; no longer JP1.2
- net D4: now also U1.P3; no longer JP1.3
- net GND: now also AVR_ISP.GND, C2.-, C3.-, IC2.GND, RESET.1, TVS1.2, U1.GND@1, U1.GND@2; no longer AVR_ISP.6, C2.2, C3.2, JP1.4, JP2.5, MIC5235.ADJ, MIC5235.GND, RESET.2
- net RAW: now also D1.A, TVS1.1, U1.RAW; no longer C2.1, JP1.5, MIC5235.EN, MIC5235.IN
- net RST: now also AVR_ISP.RST, IC1.RESET, R1.1, RESET.2, U1.RST; no longer AVR_ISP.5, IC1.PB5(NRES), JP1.1, R1.2, RESET.1
- net VCC: now also AVR_ISP.VCC, C3.+, IC2.OUT, R1.2, U1.VCC; no longer AVR_ISP.2, C3.1, JP2.4, MIC5235.OUT, R1.1
Other:
- moved on the sheet: C1, IC1, POWER, R1, R2
