File: hardware/attinier85-motherboard-pth-mk-1.0.brd (EAGLE design)
At the start: 31 x 29 mm, 11 parts, among them IC1 TINY85, U1 ATTINIER85_SHIELD

Commit message: more boards
Parts:
- removed AVR_ISP: AVR_SPI_PRG_6PTH, A_butts:2X3
- removed BATT: CR2032, A_butts:BATTCON_20MM_PTH_TOPLOAD
- removed U$1: CC-BY-SA-4.0NO-URL, A_butts:CC-BY-SA-4.0-NO-URL
- removed U1: ATTINIER85_SHIELD, A_butts:ATTINIER85_SHIELD2
- added FRAME1: FRAME-LETTERNO_PACKAGE, a_parts:DUMMY
- added JP1, JP2: M05PTH, a_parts:1X05
Connections:
- removed net MISO: AVR_ISP.1, IC1.6, U1.1
- removed net MOSI/SDA: AVR_ISP.4, IC1.5, U1.0
- removed net N$1: BATT.+, POWER.2
- removed net SCK/SCL: AVR_ISP.3, IC1.7, U1.2
- new net D1: IC1.5, JP1.4
- new net D2: IC1.6, JP1.3
- new net D5: IC1.3, JP2.3
- new net RAW: JP2.5, POWER.2
- net D3: now also IC1.7, JP1.2; no longer IC1.2, U1.4
- net D4: now also IC1.2, JP2.2; no longer IC1.3, U1.3
- net GND: now also JP1.5, JP2.4; no longer AVR_ISP.6, BATT.-, U1.GND@1, U1.GND@2
- net RST: now also JP2.1; no longer AVR_ISP.5, U1.RST
- net VCC: now also JP1.1; no longer AVR_ISP.2, U1.VCC
Routing:
- net VCC: track 39.6 -> 13.4 mm
- net N$1: track 21.0 -> 0.00 mm
- net SCK/SCL: track 17.8 -> 0.00 mm
- net RAW: track 0.00 -> 16.3 mm
- net MOSI/SDA: track 15.3 -> 0.00 mm
- net MISO: track 15.3 -> 0.00 mm
- net D2: track 0.00 -> 11.7 mm
- net D1: track 0.00 -> 11.7 mm
- net RST: track 36.2 -> 30.5 mm
- net D4: track 6.72 -> 1.80 mm
- net D3: track 6.72 -> 11.3 mm
- net D5: track 0.00 -> 1.80 mm
Other:
- board outline removed
Changed lines of the file:
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@@
 <?xml version="1.0" encoding="utf-8"?>
 <!DOCTYPE eagle SYSTEM "eagle.dtd">
-<eagle version="6.5.0">
+<eagle version="7.5.0">
 <drawing>
 <settings>
@@
 <layer number="56" name="wert" color="7" fill="1" visible="no" active="no"/>
 <layer number="57" name="tCAD" color="7" fill="1" visible="no" active="no"/>
-<layer number="90" name="Modules" color="5" fill="1" visible="yes" active="yes"/>
+<layer number="59" name="tCarbon" color="7" fill="1" visible="no" active="no"/>
+<layer number="60" name="bCarbon" color="7" fill="1" visible="no" active="no"/>
+<layer number="90" name="Modules" color="5" fill="1" visible="no" active="no"/>
 <layer number="91" name="Nets" color="2" fill="1" visible="no" active="no"/>
 <layer number="92" name="Busses" color="1" fill="1" visible="no" active="no"/>
@@
 <layer number="230" name="230bmp" color="7" fill="1" visible="yes" active="yes"/>
 <layer number="231" name="231bmp" color="7" fill="1" visible="yes" active="yes"/>
+<layer number="232" name="Eagle3D_PG2" color="7" fill="1" visible="no" active="no"/>
+<layer number="233" name="Eagle3D_PG3" color="7" fill="1" visible="no" active="no"/>
 <layer number="248" name="Housing" color="7" fill="1" visible="yes" active="yes"/>
 <layer number="249" name="Edge" color="7" fill="1" visible="yes" active="yes"/>
@@
 <pass name="Default">
 <param name="RoutingGrid" value="50mil"/>
+<param name="AutoGrid" value="1"/>
+<param name="Efforts" value="0"/>
+<param name="TopRouterVariant" value="1"/>
 <param name="tpViaShape" value="round"/>
 <param name="PrefDir.1" value="|"/>
@@
 </autorouter>
 <elements>
-<element name="U$1" library="A_butts" package="CC-BY-SA-4.0-NO-URL" value="CC-BY-SA-4.0NO-URL" x="2.2" y="24.7" rot="MR90"/>
 <element name="C1" library="A_butts" package="C025-024X044" value="0.1uF" x="22.3" y="19.58" rot="R90"/>
 <element name="IC1" library="A_butts" package="DIP08" value="TINY85" x="15.5" y="14.5" rot="R270">
@@
 <element name="RESET" library="A_butts" package="TACTILE-PTH-SIDE" value="DTS-6MM" x="25.5" y="26.9" rot="R180"/>
 <element name="R1" library="A_butts" package="RESISTOR-AXIAL-PTH-7.62MM" value="10k" x="15.5" y="21"/>
-<element name="AVR_ISP" library="A_butts" package="2X3" value="AVR_SPI_PRG_6PTH" x="15.5" y="5" rot="R180"/>
-<element name="U1" library="A_butts" package="ATTINIER85_SHIELD2" value="ATTINIER85_SHIELD" x="15.5" y="14.5"/>
 <element name="POWER" library="A_butts" package="SPDT-RA-2.54MM" value="SWITCH-SPDTPTH-RA-2.54MM" x="18" y="26.4" rot="R180"/>
-<element name="BATT" library="A_butts" package="BATTCON_20MM_PTH_TOPLOAD" value="CR2032" x="14" y="14.5" smashed="yes" rot="MR0">
-<attribute name="VALUE" x="14" y="2.6" size="0.8" layer="28" font="vector" ratio="12" rot="MR0" align="top-center"/>
-</element>
 <element name="U$4" library="A_butts" package="OSHWLOGO_TOP_0.2" value="" x="3.5" y="4" rot="MR90"/>
 <element name="U$5" library="A_butts" package="COW_SMALL_METAL" value="" x="5.5" y="5.8"/>
+<element name="FRAME1" library="a_parts" package="DUMMY" value="FRAME-LETTERNO_PACKAGE" x="-0.1" y="-0.2">
+<attribute name="DESIGNER" value="Nobody" x="-0.1" y="-0.2" size="0.5" layer="27" ratio="12" display="off"/>
+<attribute name="VERSION" value="v01" x="-0.1" y="-0.2" size="0.5" layer="27" ratio="12" display="off"/>
+</element>
+<element name="JP1" library="a_parts" package="1X05" value="M05PTH" x="0.7" y="-3.9"/>
+<element name="JP2" library="a_parts" package="1X05" value="M05PTH" x="0.7" y="-8"/>
 </elements>
 <signals>
@@
 <contactref element="IC1" pad="4"/>
 <contactref element="RESET" pad="1"/>
-<contactref element="AVR_ISP" pad="6"/>
-<contactref element="U1" pad="GND@1"/>
-<contactref element="U1" pad="GND@2"/>
-<contactref element="BATT" pad="-"/>
+<contactref element="JP1" pad="5"/>
+<contactref element="JP2" pad="4"/>
+<wire x1="22.3" y1="20.85" x2="28" y2="26.9" width="0" layer="19" extent="1-1"/>
+<wire x1="11.69" y1="10.69" x2="22.3" y2="20.85" width="0" layer="19" extent="1-1"/>
+<wire x1="10.86" y1="-3.9" x2="11.69" y2="10.69" width="0" layer="19" extent="1-1"/>
+<wire x1="8.32" y1="-8" x2="10.86" y2="-3.9" width="0" layer="19" extent="1-1"/>
 </signal>
 <signal name="VCC">
 <contactref element="R1" pad="P$2"/>
-<contactref element="AVR_ISP" pad="2"/>
 <contactref element="C1" pad="1"/>
 <contactref element="IC1" pad="8"/>
-<contactref element="U1" pad="VCC"/>
 <contactref element="POWER" pad="1"/>
 <wire x1="18" y1="26.4" x2="18" y2="22.31" width="0.6" layer="16"/>
@@
 <wire x1="19.31" y1="18.31" x2="22.3" y2="18.31" width="0.6" layer="16"/>
 <wire x1="22.3" y1="18.31" x2="23.57" y2="19.58" width="0.6" layer="16"/>
-<wire x1="23.57" y1="19.58" x2="25.5" y2="19.58" width="0.6" layer="16"/>
-<wire x1="18.04" y1="3.73" x2="21.31" y2="7" width="0.6" layer="1"/>
-<wire x1="21.31" y1="7" x2="26" y2="7" width="0.6" layer="1"/>
-<wire x1="26" y1="7" x2="28" y2="9" width="0.6" layer="1"/>
-<wire x1="28" y1="9" x2="28" y2="18" width="0.6" layer="1"/>
-<wire x1="25.5" y1="19.58" x2="26.42" y2="19.58" width="0.6" layer="1"/>
-<wire x1="26.42" y1="19.58" x2="28" y2="18" width="0.6" layer="1"/>
+<contactref element="JP1" pad="1"/>
+<wire x1="0.7" y1="-3.9" x2="19.31" y2="18.31" width="0" layer="19" extent="1-1"/>
 </signal>
 <signal name="RST">
@@
 <contactref element="R1" pad="P$1"/>
 <contactref element="RESET" pad="2"/>
-<contactref element="AVR_ISP" pad="5"/>
-<contactref element="U1" pad="RST"/>
 <wire x1="23" y1="26.9" x2="21.4" y2="26.9" width="0.3" layer="1"/>
 <wire x1="21.4" y1="26.9" x2="15.5" y2="21" width="0.3" layer="1"/>
 <wire x1="15.5" y1="21" x2="11.69" y2="21" width="0.3" layer="1"/>
 <wire x1="11.69" y1="18.31" x2="11.69" y2="21" width="0.3" layer="1"/>
-<wire x1="5.5" y1="19.58" x2="10.42" y2="19.58" width="0.3" layer="1"/>
 <wire x1="10.42" y1="19.58" x2="11.69" y2="18.31" width="0.3" layer="1"/>
 <wire x1="11.69" y1="18.31" x2="13.5" y2="16.5" width="0.3" layer="1"/>
 <wire x1="13.5" y1="16.5" x2="13.5" y2="6.81" width="0.3" layer="1"/>
-<wire x1="13.5" y1="6.81" x2="12.96" y2="6.27" width="0.3" layer="1"/>
+<contactref element="JP2" pad="1"/>
+<wire x1="0.7" y1="-8" x2="13.5" y2="6.81" width="0" layer="19" extent="1-1"/>
+</signal>
+<signal name="D5">
+<contactref element="IC1" pad="3"/>
+<wire x1="10.42" y1="14.5" x2="11.69" y2="13.23" width="0.3" layer="1"/>
+<contactref element="JP2" pad="3"/>
+<wire x1="5.78" y1="-8" x2="11.69" y2="13.23" width="0" layer="19" extent="1-1"/>
 </signal>
 <signal name="D4">
-<contactref element="IC1" pad="3"/>
-<contactref element="U1" pad="3"/>
-<wire x1="5.5" y1="14.5" x2="10.42" y2="14.5" width="0.3" layer="1"/>
-<wire x1="10.42" y1="14.5" x2="11.69" y2="13.23" width="0.3" layer="1"/>
+<contactref element="IC1" pad="2"/>
+<wire x1="10.42" y1="17.04" x2="11.69" y2="15.77" width="0.3" layer="1"/>
+<contactref element="JP2" pad="2"/>
+<wire x1="3.24" y1="-8" x2="11.69" y2="15.77" width="0" layer="19" extent="1-1"/>
 </signal>
 <signal name="D3">
-<contactref element="IC1" pad="2"/>
-<contactref element="U1" pad="4"/>
-<wire x1="5.5" y1="17.04" x2="10.42" y2="17.04" width="0.3" layer="1"/>
-<wire x1="10.42" y1="17.04" x2="11.69" y2="15.77" width="0.3" layer="1"/>
-</signal>
-<signal name="SCK/SCL">
 <contactref element="IC1" pad="7"/>
-<contactref element="AVR_ISP" pad="3"/>
-<contactref element="U1" pad="2"/>
-<wire x1="15.5" y1="6.27" x2="15.5" y2="11.96" width="0.3" layer="1"/>
 <wire x1="15.5" y1="11.96" x2="19.31" y2="15.77" width="0.3" layer="1"/>
-<wire x1="25.5" y1="17.04" x2="24.96" y2="16.5" width="0.3" layer="1"/>
 <wire x1="24.96" y1="16.5" x2="20.04" y2="16.5" width="0.3" layer="1"/>
 <wire x1="20.04" y1="16.5" x2="19.31" y2="15.77" width="0.3" layer="1"/>
-</signal>
-<signal name="MISO">
+<contactref element="JP1" pad="2"/>
+<wire x1="3.24" y1="-3.9" x2="15.5" y2="11.96" width="0" layer="19" extent="1-1"/>
+</signal>
+<signal name="D2">
 <contactref element="IC1" pad="6"/>
-<contactref element="AVR_ISP" pad="1"/>
-<contactref element="U1" pad="1"/>
-<wire x1="25.5" y1="14.5" x2="23.5" y2="12.5" width="0.3" layer="1"/>
 <wire x1="23.5" y1="12.5" x2="20.04" y2="12.5" width="0.3" layer="1"/>
 <wire x1="20.04" y1="12.5" x2="19.31" y2="13.23" width="0.3" layer="1"/>
-<wire x1="18.04" y1="6.27" x2="17.5" y2="6.81" width="0.3" layer="1"/>
 <wire x1="17.5" y1="6.81" x2="17.5" y2="11.42" width="0.3" layer="1"/>
 <wire x1="19.31" y1="13.23" x2="17.5" y2="11.42" width="0.3" layer="1"/>
-</signal>
-<signal name="MOSI/SDA">
+<contactref element="JP1" pad="3"/>
+<wire x1="5.78" y1="-3.9" x2="17.5" y2="6.81" width="0" layer="19" extent="1-1"/>
+</signal>
+<signal name="D1">
 <contactref element="IC1" pad="5"/>
-<contactref element="AVR_ISP" pad="4"/>
-<contactref element="U1" pad="0"/>
-<wire x1="25.5" y1="11.96" x2="24.23" y2="10.69" width="0.3" layer="1"/>
 <wire x1="24.23" y1="10.69" x2="19.31" y2="10.69" width="0.3" layer="1"/>
 <wire x1="16.77" y1="5" x2="16.77" y2="8.15" width="0.3" layer="16"/>
-<wire x1="15.5" y1="3.73" x2="16.77" y2="5" width="0.3" layer="16"/>
 <wire x1="19.31" y1="10.69" x2="16.77" y2="8.15" width="0.3" layer="16"/>
-</signal>
-<signal name="N$1">
-<contactref element="BATT" pad="+"/>
+<contactref element="JP1" pad="4"/>
+<wire x1="8.32" y1="-3.9" x2="16.77" y2="5" width="0" layer="19" extent="16-16"/>
+</signal>
+<signal name="RAW">
 <contactref element="POWER" pad="2"/>
-<wire x1="2.15" y1="14.5" x2="2.15" y2="19.15" width="0.6" layer="16"/>
 <wire x1="2.15" y1="19.15" x2="7.5" y2="24.5" width="0.6" layer="16"/>
 <wire x1="7.5" y1="24.5" x2="13.56" y2="24.5" width="0.6" layer="16"/>
 <wire x1="13.56" y1="24.5" x2="15.46" y2="26.4" width="0.6" layer="16"/>
+<contactref element="JP2" pad="5"/>
+<wire x1="10.86" y1="-8" x2="2.15" y2="19.15" width="0" layer="19" extent="16-16"/>
 </signal>
 </signals>
